Commit message: completed LIO_SAM

File: src/scout_bot_description/src/description/scout_bot_description.urdf (robot description, URDF)
Before this commit: robot scout_bot, 4 links, 3 joints
Links:
- added link back_camera_link, mass 0.5; collision box size=0.05 0.05 0.05; visual box size=0.05 0.05 0.05
- added link dummy_base_link; visual box size=0.001 0.001 0.001
- added link front_camera_link, mass 0.5; collision box size=0.05 0.05 0.05; visual box size=0.05 0.05 0.05
- added link gnss_link, mass 1.0; collision box size=0.2 0.1 0.05; visual box size=0.2 0.1 0.05
- added link left_camera_link, mass 0.5; collision box size=0.05 0.05 0.05; visual box size=0.05 0.05 0.05
- added link lidar_base_link, mass 0.05; collision cylinder length=0.0717 radius=0.0516; visual cylinder length=0.0717 radius=0.0516
- added link lidar_scan_link, mass 0.01; visual cylinder length=0.0717 radius=0.0516
- added link right_camera_link, mass 0.5; collision box size=0.05 0.05 0.05; visual box size=0.05 0.05 0.05
Joints:
- removed joint base_joint
- added joint back_camera_joint: type fixed, parent base_link, child back_camera_link, origin xyz=-0.5125 0 ${cam_height} rpy=0 0 ${M_PI}
- added joint base_link_joint: type fixed, parent base_link, child base_footprint, origin xyz=0.0 0.0 ${-(wheel_radius+wheel_zoff)} rpy=0 0 0
- added joint dummy_base_link_joint: type fixed, parent base_link, child dummy_base_link, origin xyz=0 0 0 rpy=0 0 0
- added joint front_camera_joint: type fixed, parent base_link, child front_camera_link, origin xyz=0.5125 0 ${cam_height} rpy=0 0 0
- added joint gnss_joint: type fixed, parent dummy_base_link, child gnss_link, origin xyz=0 0 0 rpy=0 0 0
- added joint left_camera_joint: type fixed, parent base_link, child left_camera_link, origin xyz=0 ${base_y_size/2 + cam_offset} ${cam_height} rpy=0 0 ${M_PI/2}
- added joint lida_base_link_joint: type fixed, parent base_link, child lidar_base_link, origin xyz=0.5125 0 0.05 rpy=0 0 0
- added joint lidar_scan_joint: type fixed, parent lidar_base_link, child lidar_scan_link, origin xyz=0 0 0.0377 rpy=0 0 0
- added joint right_camera_joint: type fixed, parent base_link, child right_camera_link, origin xyz=0 ${-base_y_size/2 - cam_offset} ${cam_height} rpy=0 0 ${-M_PI/2}
